File: BatteryBridge/BatteryBridge.kicad_pcb (KiCad board)
At the start: 2 copper layers, 26.4 x 52.2 mm, 24 parts, among them IC1 MAX1595EUA50+, J1 JST_PH, J2 USB_A, J3 Conn_02x20_Odd_Even, Q1 Q_PMOS_GSD, U1 MCP73832-2-OT, U2 LTC4412xS6

Commit message: Finished V1.1, added gerbers/drills
Parts:
- removed J2: USB_A, Connector_USB:USB_A_Molex_48037-2200_Horizontal
- removed J3: Conn_02x20_Odd_Even, Connector_PinSocket_2.54mm:PinSocket_2x20_P2.54mm_Vertical_SMD
- added G***: LOGO, Logo:GLogoSmall, F.Cu at (111.5, 92.4)
- added H1: MH, MountingHole:MountingHole_3.2mm_M3_Pad_Via, F.Cu at (148.3, 92.8)
- added H2: MH, MountingHole:MountingHole_2.2mm_M2_Pad_TopOnly, F.Cu at (110.0, 80.0)
- added J4: JST_BH, Connector_JST:JST_GH_SM03B-GHS-TB_1x03-1MP_P1.25mm_Horizontal, F.Cu at (119.8, 80.8)
- C1, C7, C9: value 4.7uF -> 4.7uF 0805 X5R 25V (or better)
- C2: value 10uF -> 10uF 16V X5R (or better)
- C3, C8: value 100n -> 100nF (0.1uF) 0805 X5R 10V (or better)
- C4, C5: value 2u2 -> 2.2uF 0805 X5R 25V (or better)
- C6: value 0u47 -> 0.47uF 0805 X7R 50V (or better)
- D1, D3: value GREEN -> LED GREEN CLEAR 0805 SMD
- D5: footprint Diode_THT:D_DO-15_P10.16mm_Horizontal -> Diode_THT:D_DO-41_SOD81_P7.62mm_Horizontal
- R1: value 470k -> 470k 0805 1%
- R2, R4: value 470 -> 470R 0805 1%
- R3: value 2k -> 2k 0805 1%
- moved J1 78.5 mm to (146.6, 82.3), turned to 90 degrees
- moved C5 67.5 mm to (138.1, 91.4), turned to 90 degrees
- moved C2 64.9 mm to (125.2, 90.2), turned to -90 degrees
- moved C3 62.8 mm to (132.5, 83.1)
- moved C4 62.0 mm to (134.8, 94.7), turned to 0 degrees
- moved D4 61.2 mm to (135.6, 79.5)
- moved U1 60.6 mm to (135.7, 83.1)
- moved R2 60.5 mm to (136.7, 86.6)
- moved C7 60.4 mm to (138.9, 83.1)
- moved R3 60.4 mm to (133.4, 85.9)
- moved D1 60.3 mm to (133.5, 87.9)
- moved IC1 59.6 mm to (133.8, 91.7), turned to 180 degrees
- moved C1 58.9 mm to (130.4, 83.1)
- moved R4 58.3 mm to (118.4, 90.2), turned to -90 degrees
- moved D3 55.4 mm to (116.4, 90.2), turned to -90 degrees
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Connections:
- net /VIN_RASP renamed VCOM
- net Net-(D1-K) renamed /R_LED_BAT
- net Net-(D3-A) renamed /R_LED
Routing:
- net VCOM: track 60.7 -> 16.7 mm, vias 1 -> 0
- net +5V: track 55.5 -> 42.6 mm, vias 1 -> 0
- net GND: track 15.8 -> 25.6 mm, vias 120 -> 88
- net /VBat: track 30.4 -> 24.2 mm, vias 2 -> 0
- net /BUCK_OUT: track 21.6 -> 25.5 mm
- net /GATE: track 4.83 -> 8.41 mm, vias 0 -> 2
- net /STAT_LTC: track 2.19 -> 2.70 mm
- added copper zone on In1.Cu, net GND
- added copper zone on In2.Cu, net GND
- removed copper zone on B.Cu, net GND
Other:
- board size 26.4 x 52.2 mm -> 44.2 x 18.7 mm
- copper layers 2 -> 4
- board text added: "BatteryBridge V1.1"
- board text added: "GND"
- board text added: "GND 5V VCOM"
- board text added: "VBAT"
- board text removed: "2)Bat- 1)Bat+"
- board text removed: "5V"

Commit message: Started layout labtop
Parts:
- removed C1, C7, C9: 4.7uF 0805 X5R 25V (or better), Capacitor_SMD:C_0805_2012Metric
- removed C2: 10uF 16V X5R (or better), Capacitor_SMD:C_0805_2012Metric
- removed C3, C8: 100nF (0.1uF) 0805 X5R 10V (or better), Capacitor_SMD:C_0805_2012Metric
- removed C4, C5: 2.2uF 0805 X5R 25V (or better), Capacitor_SMD:C_0805_2012Metric
- removed C6: 0.47uF 0805 X7R 50V (or better), Capacitor_SMD:C_0805_2012Metric
- removed D1, D3: LED GREEN CLEAR 0805 SMD, LED_SMD:LED_0805_2012Metric
- removed D4: SMAJ5.0A, Diode_SMD:D_SMA
- removed D5: D_Schot, Diode_THT:D_DO-41_SOD81_P7.62mm_Horizontal
- removed H1: MH, MountingHole:MountingHole_3.2mm_M3_Pad_Via
- removed H2: MH, MountingHole:MountingHole_2.2mm_M2_Pad_TopOnly
- removed IC1: MAX1595EUA50+, Footprints:SOP65P490X110-8N
- removed J1: JST_PH, Connector_JST:JST_PH_S2B-PH-SM4-TB_1x02-1MP_P2.00mm_Horizontal
- removed J4: JST_BH, Connector_JST:JST_GH_SM03B-GHS-TB_1x03-1MP_P1.25mm_Horizontal
- removed Q1: Q_PMOS_GSD, Package_TO_SOT_SMD:SOT-23
- removed R1: 470k 0805 1%, Resistor_SMD:R_0805_2012Metric
- removed R2, R4: 470R 0805 1%, Resistor_SMD:R_0805_2012Metric
- removed R3: 2k 0805 1%, Resistor_SMD:R_0805_2012Metric
- removed U1: MCP73832-2-OT, Package_TO_SOT_SMD:SOT-23-5
- removed U2: LTC4412xS6, Package_TO_SOT_SMD:TSOT-23-6
- added C201: 10u, Capacitor_SMD:C_0805_2012Metric, F.Cu at (129.0, 97.5)
- added C202: 2n2, Capacitor_SMD:C_0805_2012Metric, F.Cu at (84.8, 78.9)
- added C203: 10u, Capacitor_SMD:C_0805_2012Metric, B.Cu at (80.4, 82.1)
- added C204: 100p, Capacitor_SMD:C_0805_2012Metric, F.Cu at (79.8, 80.4)
- added C205: 22u, Capacitor_SMD:C_0805_2012Metric, F.Cu at (132.6, 99.6)
- added C206: 100n, Capacitor_SMD:C_0805_2012Metric, F.Cu at (132.2, 91.8)
- added C207: 22u, Capacitor_SMD:C_0805_2012Metric, F.Cu at (132.6, 97.5)
- added C208: 100n, Capacitor_SMD:C_0805_2012Metric, F.Cu at (84.7, 81.0)
- added C209: 1n8, Capacitor_SMD:C_0805_2012Metric, F.Cu at (137.6, 78.9)
- added C210: 10u, Capacitor_SMD:C_0805_2012Metric, F.Cu at (143.8, 85.9)
- added C211: 47p, Capacitor_SMD:C_0805_2012Metric, F.Cu at (137.5, 83.0)
- added C212: 22u, Capacitor_SMD:C_1210_3225Metric, F.Cu at (90.4, 93.1)
- added C213: 1n, Capacitor_SMD:C_0805_2012Metric, F.Cu at (139.1, 88.8)
- added C214: 22u, Capacitor_SMD:C_1210_3225Metric, F.Cu at (94.1, 93.1)
- added C215: 20SVPF120M, Footprints:16SVF180M, F.Cu at (83.8, 91.4)
- added C216: 100u, Capacitor_SMD:C_0805_2012Metric, F.Cu at (126.4, 88.8)
- added C217: 100u, Capacitor_SMD:C_0805_2012Metric, F.Cu at (128.5, 88.8)
- added C301: 100n, Capacitor_SMD:C_0805_2012Metric, B.Cu at (132.5, 84.5)
- added C302: 4.7u, Capacitor_SMD:C_0805_2012Metric, B.Cu at (130.3, 84.5)
- added C303: 4.7u, Capacitor_SMD:C_0805_2012Metric, B.Cu at (139.0, 84.4)
- added C401: 4.7u, Capacitor_SMD:C_0805_2012Metric, F.Cu at (107.3, 90.0)
- added C402: 100n, Capacitor_SMD:C_0805_2012Metric, F.Cu at (105.2, 90.0)
- added C403: 10u, Capacitor_SMD:C_0805_2012Metric, F.Cu at (98.7, 93.9)
- added C404: 4.7u, Capacitor_SMD:C_0805_2012Metric, F.Cu at (123.3, 89.7)
- added C405: 100n, Capacitor_SMD:C_0805_2012Metric, F.Cu at (121.1, 89.7)
- added C406: 10u, Capacitor_SMD:C_0805_2012Metric, F.Cu at (114.6, 93.6)
- added D201: PDS1040-13, Footprints:PDS104013, F.Cu at (76.0, 92.4)
- added D202: B320-13-F, Diode_SMD:D_SMC, F.Cu at (130.3, 83.5)
- added D301: SMAJ5.0A, Diode_SMD:D_SMA, B.Cu at (127.6, 84.3)
- added D302: GREEN, LED_SMD:LED_0805_2012Metric, B.Cu at (133.5, 79.6)
- added D401: 1N5819, Diode_THT:D_DO-41_SOD81_P7.62mm_Horizontal, F.Cu at (99.1, 86.2)
- added D402: GREEN, LED_SMD:LED_0805_2012Metric, F.Cu at (105.8, 92.7)
- added D403: 1N5819, Diode_THT:D_DO-41_SOD81_P7.62mm_Horizontal, F.Cu at (122.3, 86.0)
- added D404: GREEN, LED_SMD:LED_0805_2012Metric, F.Cu at (122.0, 92.6)
- added H101: MH, MountingHole:MountingHole_3.2mm_M3_Pad_Via, F.Cu at (148.2, 92.7)
- added H102: MH, MountingHole:MountingHole_2.2mm_M2_Pad_TopOnly, F.Cu at (110.0, 80.0)
- added IC201: SI4114DY-T1-GE3, Footprints:SOIC127P600X175-8N, F.Cu at (75.9, 83.9)
- added J101: JST_BH, Connector_JST:JST_GH_SM03B-GHS-TB_1x03-1MP_P1.25mm_Horizontal, F.Cu at (118.2, 80.9)
- added J102: JST_BH, Connector_JST:JST_GH_SM03B-GHS-TB_1x03-1MP_P1.25mm_Horizontal, F.Cu at (102.7, 81.1)
- added J301: JST_PH, Connector_JST:JST_PH_S2B-PH-SM4-TB_1x02-1MP_P2.00mm_Horizontal, B.Cu at (146.5, 82.7)
- added L201: 4.7u, Footprints:HCM1A0805-4R7-R, F.Cu at (138.9, 94.9)
- added L202: 2u2, Footprints:DR125-2R2-R, B.Cu at (89.4, 84.3)
- added L203: 1u, Footprints:PA4341.102NLT, F.Cu at (148.0, 84.5)
- added Q201: SI3460DDV-T1-GE3, Package_SO:TSOP-6_1.65x3.05mm_P0.95mm, F.Cu at (141.4, 82.3)
- added Q401: BSS84LT1G, Package_TO_SOT_SMD:SOT-23, F.Cu at (101.9, 93.9)
- added Q402: BSS84LT1G, Package_TO_SOT_SMD:SOT-23, F.Cu at (118.0, 93.6)
- added R201: 4M7, Resistor_SMD:R_0805_2012Metric, F.Cu at (86.3, 83.9)
- added R202: 23k2, Resistor_SMD:R_0805_2012Metric, F.Cu at (81.9, 80.4)
- added R203: 107k, Resistor_SMD:R_0805_2012Metric, B.Cu at (77.0, 85.1)
- added R204: 11k8, Resistor_SMD:R_0805_2012Metric, B.Cu at (76.1, 82.3)
- added R205: 1M, Resistor_SMD:R_0805_2012Metric, F.Cu at (142.7, 88.7)
- added R206: 17k4, Resistor_SMD:R_0805_2012Metric, F.Cu at (137.5, 80.9)
- added R207: 34k8, Resistor_SMD:R_0805_2012Metric, F.Cu at (131.7, 88.8)
- added R208: 11k, Resistor_SMD:R_0805_2012Metric, F.Cu at (135.2, 88.8)
- added R301: 2k, Resistor_SMD:R_0805_2012Metric, B.Cu at (133.4, 81.7)
- added R302: 470R, Resistor_SMD:R_0805_2012Metric, B.Cu at (136.6, 80.7)
- added R401: 470k, Resistor_SMD:R_0805_2012Metric, F.Cu at (98.6, 90.0)
- added R402: 470R, Resistor_SMD:R_0805_2012Metric, F.Cu at (105.8, 94.7)
- added R403: 470k, Resistor_SMD:R_0805_2012Metric, F.Cu at (114.6, 89.7)
- added R404: 470R, Resistor_SMD:R_0805_2012Metric, F.Cu at (121.9, 94.7)
- added U201: AP63205WU, Package_TO_SOT_SMD:TSOT-23-6, F.Cu at (130.6, 94.6)
- added U202: LTC3872HTS8-1-TRMPBF, Package_TO_SOT_SMD:TSOT-23-8_HandSoldering, F.Cu at (82.1, 83.9)
- added U203: LTC3872HTS8-1-TRMPBF, Package_TO_SOT_SMD:TSOT-23-8_HandSoldering, F.Cu at (139.3, 85.9)
- added U301: MCP73832-2-OT, Package_TO_SOT_SMD:SOT-23-5, B.Cu at (135.6, 84.5)
- added U401: LTC4412xS6, Package_TO_SOT_SMD:TSOT-23-6, F.Cu at (101.9, 90.0)
- added U402: LTC4412xS6, Package_TO_SOT_SMD:TSOT-23-6, F.Cu at (117.9, 89.7)
- moved G*** 29.0 mm to (110.3, 121.4)
Routing:
- net +BATT: track 0.00 -> 91.4 mm, vias 0 -> 4
- net +12V: track 0.00 -> 52.1 mm, vias 0 -> 2
- net BUCK_OUT12: track 0.00 -> 44.5 mm, vias 0 -> 1
- net /BUCK_OUT: track 25.5 -> 0.00 mm
- net VDD: track 0.00 -> 25.0 mm, vias 0 -> 2
- net /VBat: track 24.2 -> 0.00 mm
- net BUCK_OUT: track 0.00 -> 23.8 mm
- net Net-(D201-A1): track 0.00 -> 21.4 mm, vias 0 -> 2
- net /Converters/SW_D: track 0.00 -> 20.8 mm
- net /Converters/VREF5: track 0.00 -> 19.6 mm
- net Net-(IC201-G): track 0.00 -> 13.2 mm
- net GND: track 25.6 -> 14.7 mm, vias 88 -> 14
- net Net-(U201-SW): track 0.00 -> 8.60 mm
- net Net-(U202-ITH): track 0.00 -> 8.58 mm
- net /GATE: track 8.41 -> 0.00 mm, vias 2 -> 0
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- added copper zone on B.Cu, net GND
- removed copper zone on F.Cu, net +5V
- removed copper zone on F.Cu, net /VBat
Other:
- board size 44.2 x 18.7 mm -> 79.7 x 23.6 mm

Commit message: Finished v1.2, added gerbers
Parts:
- added Q404: MMBT3906-7-F, Package_TO_SOT_SMD:SOT-23-3, B.Cu at (107.5, 93.9)
- added Q405: MMBT2222A, Package_TO_SOT_SMD:SOT-23-3, B.Cu at (101.2, 90.5)
- added R405: 1k, Resistor_SMD:R_0805_2012Metric, B.Cu at (104.3, 93.7)
- added R406: 10k, Resistor_SMD:R_0805_2012Metric, B.Cu at (101.2, 94.3)
- added R407: 5k1, Resistor_SMD:R_0805_2012Metric, B.Cu at (104.3, 89.7)
- added R408: 100k, Resistor_SMD:R_0805_2012Metric, B.Cu at (107.6, 90.7)
- IC201: moved to B.Cu
- R203, R204: moved to F.Cu
- moved G*** 40.9 mm to (94.1, 83.9), turned to 0 degrees
- moved C401 9.92 mm to (98.0, 93.5), turned to 90 degrees
- moved R401 9.87 mm to (107.4, 94.4), turned to 180 degrees
- moved C403 9.08 mm to (106.8, 89.7), turned to -90 degrees
- moved D402 8.08 mm to (98.3, 89.8), turned to -90 degrees
- moved R402 7.39 mm to (100.3, 89.8), turned to -90 degrees
- moved C402 6.14 mm to (100.2, 93.5), turned to 90 degrees
- moved Q401 4.43 mm to (103.5, 89.8), turned to 180 degrees
- moved C209 3.93 mm to (134.4, 81.2)
- moved U401 3.85 mm to (103.4, 93.5), turned to 0 degrees
- moved C211 3.85 mm to (134.4, 85.2), turned to 180 degrees
- moved R206 3.85 mm to (134.4, 83.2), turned to 0 degrees
- moved C203 3.30 mm to (82.9, 84.3), turned to 180 degrees
- moved IC201 2.99 mm to (76.5, 86.8)
- moved R404 2.45 mm to (119.8, 93.5), turned to 90 degrees
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Connections:
- net Net-(D201-A1) renamed /Converters/sw_LTC12
- net Net-(U201-SW) renamed /Converters/sw_AP63
- U401 pad 6: +12V -> /PowerPathController/Sense
Routing:
- net +BATT: track 91.4 -> 4.62 mm, vias 4 -> 11
- net +12V: track 52.1 -> 13.2 mm, vias 2 -> 6
- net BUCK_OUT12: track 44.5 -> 11.0 mm, vias 1 -> 0
- net VDD: track 25.0 -> 0.00 mm, vias 2 -> 0
- net BUCK_OUT: track 23.8 -> 0.00 mm
- net /Converters/sw_LTC12: track 21.4 -> 0.00 mm, vias 2 -> 11
- net /Converters/SW_D: track 20.8 -> 0.00 mm
- net GND: track 14.7 -> 0.00 mm, vias 14 -> 82
- net +5V: track 42.5 -> 51.9 mm
- net /Converters/VREF5: track 19.6 -> 10.3 mm, vias 0 -> 2
- net /Converters/sw_AP63: track 8.60 -> 0.00 mm
- net Net-(Q201-G): track 4.66 -> 11.0 mm, vias 0 -> 2
- net Net-(IC201-G): track 13.2 -> 7.02 mm, vias 0 -> 1
- net Net-(Q404-B): track 0.00 -> 5.74 mm
- net /PowerPathController/Sense: track 0.00 -> 5.73 mm, vias 0 -> 1
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- added copper zone on B.Cu, net +12V
- added copper zone on F.Cu, net +12V
- added copper zone on In2.Cu, net +12V
- added copper zone on B.Cu, net +5V
- added copper zone on B.Cu, net +BATT
- added copper zone on F.Cu, net +BATT
- added copper zone on In2.Cu, net +BATT
- added copper zone on F.Cu, net /Converters/SW_D
- added copper zone on F.Cu, net /Converters/VREF5
- added copper zone on F.Cu, net /Converters/sw_AP63
- added copper zone on B.Cu, net /Converters/sw_LTC12
- added copper zone on F.Cu, net /Converters/sw_LTC12
- added copper zone on F.Cu, net BUCK_OUT
- added copper zone on F.Cu, net BUCK_OUT12
- added copper zone on In3.Cu, net GND
- added copper zone on In4.Cu, net GND
- added copper zone on F.Cu, net VDD
- removed copper zone on In2.Cu, net GND
Other:
- copper layers 4 -> 6
- board text added: "12V"
- board text added: "5V"
- board text added: "BatteryBridge V1.2"
- board text added: "VCOM"
- board text added: "VDD"
- board text added: "VREF"
- board text removed: "BatteryBridge V1.1"
- board text removed: "GND 5V VCOM"
