File: BatteryBridge/BatteryBridge.kicad_sch (KiCad schematic)
At the start: 24 parts, among them IC1 MAX1595EUA50+, J1 JST_PH, J2 USB_A, J3 Conn_02x20_Odd_Even, Q1 Q_PMOS_GSD, U1 MCP73832-2-OT, U2 LTC4412xS6

Commit message: Finished V1.1, added gerbers/drills
Parts:
- removed J2: USB_A, Connector_USB:USB_A_Molex_48037-2200_Horizontal, symbol Connector:USB_A
- removed J3: Conn_02x20_Odd_Even, Connector_PinSocket_2.54mm:PinSocket_2x20_P2.54mm_Vertical_SMD, symbol Connector_Generic:Conn_02x20_Odd_Even
- added H1: MH, MountingHole:MountingHole_3.2mm_M3_Pad_Via, symbol Mechanical:MountingHole_Pad
- added H2: MH, MountingHole:MountingHole_2.2mm_M2_Pad_TopOnly, symbol Mechanical:MountingHole_Pad
- added J4: JST_BH, Connector_JST:JST_GH_SM03B-GHS-TB_1x03-1MP_P1.25mm_Horizontal, symbol Connector_Generic_MountingPin:Conn_01x03_MountingPin
- C1, C7, C9: value 4.7uF -> 4.7uF 0805 X5R 25V (or better)
- C2: value 10uF -> 10uF 16V X5R (or better)
- C3, C8: value 100n -> 100nF (0.1uF) 0805 X5R 10V (or better)
- C4, C5: value 2u2 -> 2.2uF 0805 X5R 25V (or better)
- C6: value 0u47 -> 0.47uF 0805 X7R 50V (or better)
- D1, D3: value GREEN -> LED GREEN CLEAR 0805 SMD
- D5: footprint Diode_THT:D_DO-15_P10.16mm_Horizontal -> Diode_THT:D_DO-41_SOD81_P7.62mm_Horizontal
- R1: value 470k -> 470k 0805 1%
- R2, R4: value 470 -> 470R 0805 1%
- R3: value 2k -> 2k 0805 1%
Connections:
- net +5V: now also J4.2 (Pin_2)
- net GND: now also J4.3 (Pin_3), J4.MP (MountPin)
- net R_LED_BAT: now reaches D1.1 (K), R2.1
- net R_LED: now reaches D3.2 (A), R4.2
- net VIN_RASP renamed VCOM
- net VCOM: now also J4.1 (Pin_1)
- no-connect marks 40 -> 2
Other:
- note removed: "Connectors"
- note removed: "Power connector (5V IN)"
- note removed: "Raspberry Pi connector (LOAD)"

Commit message: Finished schematic and component selection
Parts:
- removed C1, C7, C9: 4.7uF 0805 X5R 25V (or better), Capacitor_SMD:C_0805_2012Metric, symbol Device:C
- removed C2: 10uF 16V X5R (or better), Capacitor_SMD:C_0805_2012Metric, symbol Device:C
- removed C3, C8: 100nF (0.1uF) 0805 X5R 10V (or better), Capacitor_SMD:C_0805_2012Metric, symbol Device:C
- removed C4, C5: 2.2uF 0805 X5R 25V (or better), Capacitor_SMD:C_0805_2012Metric, symbol Device:C
- removed C6: 0.47uF 0805 X7R 50V (or better), Capacitor_SMD:C_0805_2012Metric, symbol Device:C
- removed D1, D3: LED GREEN CLEAR 0805 SMD, LED_SMD:LED_0805_2012Metric, symbol Device:LED
- removed D4: SMAJ5.0A, Diode_SMD:D_SMA, symbol Diode:SMAJ5.0A
- removed D5: D_Schot, Diode_THT:D_DO-41_SOD81_P7.62mm_Horizontal, symbol Device:D_Schottky
- removed IC1: MAX1595EUA50+, Footprints:SOP65P490X110-8N, symbol MAX1595EUA50+:MAX1595EUA50+
- removed J1: JST_PH, Connector_JST:JST_PH_S2B-PH-SM4-TB_1x02-1MP_P2.00mm_Horizontal, symbol Connector_Generic_MountingPin:Conn_01x02_MountingPin
- removed Q1: Q_PMOS_GSD, Package_TO_SOT_SMD:SOT-23, symbol Device:Q_PMOS_GSD
- removed R1: 470k 0805 1%, Resistor_SMD:R_0805_2012Metric, symbol Device:R
- removed R2, R4: 470R 0805 1%, Resistor_SMD:R_0805_2012Metric, symbol Device:R
- removed R3: 2k 0805 1%, Resistor_SMD:R_0805_2012Metric, symbol Device:R
- removed U1: MCP73832-2-OT, Package_TO_SOT_SMD:SOT-23-5, symbol Battery_Management:MCP73832-2-OT
- removed U2: LTC4412xS6, Package_TO_SOT_SMD:TSOT-23-6, symbol Power_Management:LTC4412xS6
- added J102: JST_BH, Connector_JST:JST_GH_SM03B-GHS-TB_1x03-1MP_P1.25mm_Horizontal, symbol Connector_Generic_MountingPin:Conn_01x03_MountingPin
- renumbered H1 to H101, H2 to H102, J4 to J101
Connections:
- net GND: now also J102.MP (MountPin)
- new net +12V: J102.1 (Pin_1)
- new net VDD: J102.2 (Pin_2)
- no-connect marks 2 -> 3
Other:
- added sheet BatteryCharger (BatCharge.kicad_sch)
- added sheet Converters (ConvertersBat.kicad_sch)
- added sheet PowerPathController (PPController.kicad_sch)
- note added: "INPUT CONNECTORS"
- note added: "[2] CONVERTERS"
- note added: "[3] Battery Charger"
- note added: "[4] Power Path Controllers"
- note removed: "Battery charger circuit"
- note removed: "Buck converter circuit"
- note removed: "ChargeCurrent (IReg)=1000V/RProg=1000V/2=500mA Rprog=kOhms Ireg=milliamps"
- note removed: "DATASHEET: Place capacitors as close as possible to MAX1595"
- note removed: "MAX CURRENT DELIVERY: 125mA"
- note removed: "PLACE C8 AND C9 CLOSE TO VIN"
- note removed: "PLACE NEAR VDD"
- note removed: "Powerpath controller circuit"
- note removed: "V(ripple)=Iout/(2*fosc*Cout) =0.125A/(2*1.000.000MHz*0.0022F)=0.00028V Capacitor values gives ~35mV ripples"
- moved on the sheet: H101, H102, J101

Commit message: Started layout labtop
Changed lines of the file:
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@@
+	)
+	(junction
+		(at 248.92 127)
+		(diameter 0)
+		(color 0 0 0 0)
 	)
 	(junction
@@
 	(wire
 		(pts
-			(xy 248.92 125.73) (xy 248.92 134.62)
+			(xy 248.92 125.73) (xy 248.92 127)
 		)
 		(stroke
@@
 		(pts
 			(xy 251.46 125.73) (xy 251.46 128.27)
+		)
+		(stroke
+			(width 0)
+			(type default)
+		)
+	)
+	(wire
+		(pts
+			(xy 248.92 127) (xy 248.92 134.62)
 		)
 		(stroke
@@
 					(unit 1)
 				)
+			)
+		)
+	)
+	(symbol
+		(lib_id "power:PWR_FLAG")
+		(at 248.92 127 90)
+		(unit 1)
+		(exclude_from_sim no)
+		(in_bom yes)
+		(on_board yes)
+		(dnp no)
+		(property "Reference" "#FLG01"
+			(at 247.015 127 0)
+			(effects
+				(font
+					(size 1.27 1.27)
+				)
+				(hide yes)
+			)
+		)
+		(property "Value" "PWR_FLAG"
+			(at 245.11 126.9999 90)
+			(effects
+				(font
+					(size 1.27 1.27)
+				)
+				(justify left)
+			)
+		)
+		(property "Footprint" ""
+			(at 248.92 127 0)
+			(effects
+				(font
+					(size 1.27 1.27)
+				)
+				(hide yes)
+			)
+		)
+		(property "Datasheet" "~"
+			(at 248.92 127 0)
+			(effects
+				(font
+					(size 1.27 1.27)
+				)
+				(hide yes)
+			)
+		)
+		(property "Description" "Special symbol for telling ERC where power comes from"
+			(at 248.92 127 0)
+			(effects
+				(font
+					(size 1.27 1.27)
+				)
+				(hide yes)
+			)
+		)
+		(pin "1"
+		)
+		(instances
+			(project "BatteryBridge"
+				(path "/5e95e951-7871-40f6-afbb-b8706a3712de"
+					(reference "#FLG01")
+					(unit 1)
+				)
