File: BatteryBridge/ConvertersBat.kicad_sch (KiCad schematic)
At the start: 35 parts, among them IC201 SI4114DY-T1-GE3, Q201 SI3460DDV-T1-GE3, U201 AP63205WU, U202 LTC3872HTS8-1-TRMPBF, U203 LTC3872HTS8-1-TRMPBF

Commit message: Started layout labtop
Parts:
- L202: footprint Footprints:DR125-2R2 -> Footprints:DR125-2R2-R
- Q201: footprint Footprints:SOT95P284X110-6N -> Package_SO:TSOP-6_1.65x3.05mm_P0.95mm
Changed lines of the file:
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@@
 		)
 	)
-	(label "BUCK_OUT12"
-		(at 147.32 139.7 0)
+	(label "RUN{slash}SS_5V"
+		(at 105.41 54.61 90)
 		(fields_autoplaced yes)
 		(effects
@@
 		)
 	)
-	(label "BUCK_OUT"
-		(at 229.87 53.34 180)
+	(label "RUN{slash}SS_12V"
+		(at 73.66 158.75 0)
 		(fields_autoplaced yes)
 		(effects
@@
 				(size 1.27 1.27)
 			)
-			(justify right bottom)
+			(justify left bottom)
 		)
 	)
-	(label "RUN{slash}SS_5V"
-		(at 105.41 54.61 90)
+	(label "RUN{slash}SS_12V"
+		(at 24.13 144.78 90)
 		(fields_autoplaced yes)
 		(effects
@@
 		)
 	)
-	(label "RUN{slash}SS_12V"
-		(at 73.66 158.75 0)
+	(label "BUCK_OUT12"
+		(at 48.26 125.73 0)
 		(fields_autoplaced yes)
 		(effects
@@
 		)
 	)
-	(label "BUCK_OUT"
-		(at 132.08 36.83 90)
+	(label "RUN{slash}SS_5V"
+		(at 156.21 73.66 0)
 		(fields_autoplaced yes)
 		(effects
@@
 		)
 	)
-	(label "RUN{slash}SS_12V"
-		(at 24.13 144.78 90)
+	(label "SW_D"
+		(at 189.23 52.07 0)
 		(fields_autoplaced yes)
 		(effects
@@
 		)
 	)
-	(label "BUCK_OUT12"
-		(at 48.26 125.73 0)
+	(global_label "BUCK_OUT12"
+		(shape input)
+		(at 167.64 139.7 90)
 		(fields_autoplaced yes)
 		(effects
@@
 				(size 1.27 1.27)
 			)
-			(justify left bottom)
+			(justify left)
+		)
+		(property "Intersheetrefs" "${INTERSHEET_REFS}"
+			(at 167.64 124.5591 90)
+			(effects
+				(font
+					(size 1.27 1.27)
+				)
+				(justify left)
+				(hide yes)
+			)
 		)
 	)
-	(label "RUN{slash}SS_5V"
-		(at 156.21 73.66 0)
+	(global_label "BUCK_OUT"
+		(shape input)
+		(at 132.08 36.83 90)
 		(fields_autoplaced yes)
 		(effects
@@
 				(size 1.27 1.27)
 			)
-			(justify left bottom)
+			(justify left)
+		)
+		(property "Intersheetrefs" "${INTERSHEET_REFS}"
+			(at 132.08 24.1081 90)
+			(effects
+				(font
+					(size 1.27 1.27)
+				)
+				(justify left)
+				(hide yes)
+			)
 		)
 	)
-	(label "SW_D"
-		(at 189.23 52.07 0)
+	(global_label "BUCK_OUT"
+		(shape input)
+		(at 229.87 53.34 90)
 		(fields_autoplaced yes)
 		(effects
@@
 				(size 1.27 1.27)
 			)
-			(justify left bottom)
+			(justify left)
+		)
+		(property "Intersheetrefs" "${INTERSHEET_REFS}"
+			(at 229.87 40.6181 90)
+			(effects
+				(font
+					(size 1.27 1.27)
+				)
+				(justify left)
+				(hide yes)
+			)
 		)
 	)
@@
 			)
 		)
-		(property "Footprint" "Footprints:SOT95P284X110-6N"
+		(property "Footprint" "Package_SO:TSOP-6_1.65x3.05mm_P0.95mm"
 			(at 199.39 150.8 0)
 			(effects
@@
 			)
 		)
-		(property "Footprint" "Footprints:DR125-2R2"
+		(property "Footprint" "Footprints:DR125-2R2-R"
 			(at 81.28 128.27 0)
 			(effects

Commit message: Finished v1.2, added gerbers
Connections:
- net sw_AP63: now reaches C206.1, L201.1, U201.5 (SW)
- net sw_LTC12: now reaches D201.1 (A1), D201.2 (A2), IC201.5 (D_1), IC201.6 (D_2), IC201.7 (D_3), IC201.8 (D_4), L202.2, U202.8 (SW)
Changed lines of the file:
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@@
+		)
+	)
+	(label "sw_LTC12"
+		(at 93.98 139.7 0)
+		(fields_autoplaced yes)
+		(effects
+			(font
+				(size 1.27 1.27)
+			)
+			(justify left bottom)
 		)
 	)
@@
 		(fields_autoplaced yes)
 		(effects
+			(font
+				(size 1.27 1.27)
+			)
+			(justify left bottom)
+		)
+	)
+	(label "sw_AP63"
+		(at 53.34 48.26 90)
+		(fields_autoplaced yes)
+		(effects
